Commit message: Updateing robot model.

File: src/tfr_description/xacro/model_base.xacro (robot description, xacro)
@@ -73,5 +73,5 @@
     <parent link="base_link" />
     <child link="tread_left_link" />
-    <origin xyz="0 ${tread_spacing / 2 + tread_width / 2} 0" />
+    <origin xyz="${2*itom} ${tread_spacing / 2 + tread_width / 2} ${3*itom}" />
   </joint>
   <link name="tread_right_link">
@@ -90,5 +90,5 @@
     <parent link="base_link" />
     <child link="tread_right_link" />
-    <origin xyz="0 ${-tread_spacing / 2 - tread_width / 2} 0" />
+    <origin xyz="${2*itom} ${-tread_spacing / 2 - tread_width / 2} ${3*itom}" />
   </joint>
   <link name="tread_left_front_link">
@@ -109,5 +109,5 @@
     <parent link="tread_left_link" />
     <child link="tread_left_front_link" />
-    <origin xyz="${intertread_length / 2} 0 ${-1.38*itom}" />
+    <origin xyz="${(intertread_length / 2)} 0 ${-3*itom}" />
   </joint>
   <link name="tread_left_rear_link">
@@ -128,5 +128,5 @@
     <parent link="tread_left_link" />
     <child link="tread_left_rear_link" />
-    <origin xyz="${-intertread_length / 2} 0 ${-1.38*itom}" />
+    <origin xyz="${(-intertread_length / 2)} 0 ${-3*itom}" />
   </joint>
   <link name="tread_right_front_link">
@@ -147,5 +147,5 @@
     <parent link="tread_right_link" />
     <child link="tread_right_front_link" />
-    <origin xyz="${intertread_length / 2} 0 ${-1.38*itom}" />
+    <origin xyz="${(intertread_length / 2)} 0 ${-3*itom}" />
   </joint>
   <link name="tread_right_rear_link">
@@ -166,5 +166,5 @@
     <parent link="tread_right_link" />
     <child link="tread_right_rear_link" />
-    <origin xyz="${-intertread_length / 2} 0 ${-1.38*itom}" />
+    <origin xyz="${(-intertread_length / 2)} 0 ${-3*itom}" />
   </joint>
   <link name="front_right_slope_link">

File: src/tfr_description/xacro/model_constants.xacro (robot description, xacro)
@@ -10,16 +10,16 @@
   <!-- Drivebase parameters -->
   <xacro:property name="base_length" value="${50*itom}" />
-  <xacro:property name="tube_width" value="${2*itom}" />
-  <xacro:property name="drivebase_beam_width" value="${11.5*itom}" />
-  <xacro:property name="drivebase_front_beam_height" value="${4*itom}" />
-  <xacro:property name="drivebase_total_height" value="${6*itom}" />
+  <xacro:property name="tube_width" value="${2.25*itom}" />
+  <xacro:property name="drivebase_beam_width" value="${13.75*itom}" />
+  <xacro:property name="drivebase_front_beam_height" value="${2*itom}" />
+  <xacro:property name="drivebase_total_height" value="${4.5*itom}" />
   <!-- Drivetrain parameters -->
-  <xacro:property name="tread_end_radius" value="${(15.5/2)*itom}" />
-  <xacro:property name="tread_mid_height" value="${19*itom}" />
-  <xacro:property name="tread_mid_length" value="${24*itom}" />
-  <xacro:property name="tread_width" value="${6*itom}" />
-  <xacro:property name="tread_spacing" value="${16*itom}" />
-  <xacro:property name="intertread_length" value="${39*itom}" />
-  <xacro:property name="tread_slope_length" value="${11*itom}" />
+  <xacro:property name="tread_end_radius" value="${6*itom}" />
+  <xacro:property name="tread_mid_height" value="${18.5*itom}" />
+  <xacro:property name="tread_mid_length" value="${14*itom}" />
+  <xacro:property name="tread_width" value="${4*itom}" />
+  <xacro:property name="tread_spacing" value="${20*itom}" />
+  <xacro:property name="intertread_length" value="${32*itom}" />
+  <xacro:property name="tread_slope_length" value="${1*itom}" />
   <!-- Bin parameters -->
   <!-- Length of top of bin, length of bottom is 13.86 -->

Commit message: Update model_base.xacro

File: src/tfr_description/xacro/model_base.xacro (robot description, xacro)
@@ -14,5 +14,5 @@
         <box size="${base_length} ${tube_width} ${drivebase_total_height}"/>
       </geometry>
-      <origin xyz="0 ${drivebase_beam_width / 2 + tube_width / 2} 0" />
+      <origin xyz="0 ${drivebase_beam_width / 2 + tube_width / 2} 0.15" />
     </visual>
     <visual>

Commit message: Update model_base.xacro

File: src/tfr_description/xacro/model_base.xacro (robot description, xacro)
@@ -4,5 +4,5 @@
   <link name="base_footprint" />
   <joint name="base_footprint_joint" type="fixed">
-    <origin xyz="0 0 0.017" rpy="0 0 0" />
+    <origin xyz="0 0 0.15" rpy="0 0 0" />
     <parent link="base_footprint" />
     <child link="base_link" />

Commit message: Adding resized model to master branch

File: src/tfr_description/xacro/model_base.xacro (robot description, xacro)
@@ -4,5 +4,5 @@
   <link name="base_footprint" />
   <joint name="base_footprint_joint" type="fixed">
-    <origin xyz="0 0 0.15" rpy="0 0 0" />
+    <origin xyz="0 0 0.017" rpy="0 0 0" />
     <parent link="base_footprint" />
     <child link="base_link" />
@@ -14,5 +14,5 @@
         <box size="${base_length} ${tube_width} ${drivebase_total_height}"/>
       </geometry>
-      <origin xyz="0 ${drivebase_beam_width / 2 + tube_width / 2} 0.15" />
+      <origin xyz="0 ${drivebase_beam_width / 2 + tube_width / 2} 0" />
     </visual>
     <visual>
@@ -275,5 +275,5 @@
     <inertial>
       <mass value="1.0" />
-      <inertia ixx="1.0" ixy="0.0" ixz="0.0" iyy="1.0" iyz="0.0" izz="1.0"/>
+      <inertia ixx="0.0" ixy="0.0" ixz="0.0" iyy="0.0" iyz="0.0" izz="0.0"/>
     </inertial>
   </link>
@@ -373,29 +373,5 @@
     <parent link="bin_back" />
     <child link="bin_slope" />
-    <origin xyz="0 0 ${(12-9.88) * itom}" rpy="0 ${-pi/4} 0"/>
-  </joint>
-  <link name="bin_slope_2" >
-    <visual>
-      <geometry>
-        <box size="${0.125*itom} ${bin_width} ${bin_height*sqrt2}" />
-      </geometry>
-      <origin xyz="${bin_back_offset} 0 0"/>
-    </visual>
-    <collision>
-      <geometry>
-        <box size="${0.125*itom} ${bin_width} ${bin_height*sqrt2}" />
-      </geometry>
-      <origin xyz=" ${bin_back_offset}  0 0"/>
-    </collision>
-    <!-- test -->
-    <inertial>
-      <mass value="1.0" />
-      <inertia ixx="1.0" ixy="0.0" ixz="0.0" iyy="1.0" iyz="0.0" izz="1.0"/>
-    </inertial>
-  </link>
-  <joint name="bin_slope_2_joint" type="fixed">
-    <parent link="bin_back" />
-    <child link="bin_slope_2" />
-    <origin xyz="0  0 ${(12-9.88) * itom}" rpy="0 -0.105 0"/>
+    <origin xyz="0 0 ${-0.30* itom}" rpy="0 ${-pi/4} 0"/>
   </joint>
 </robot>

Commit message: Arm digging and model updates with Su, Melody, and Chris

File: src/tfr_description/xacro/model_base.xacro (robot description, xacro)
@@ -14,5 +14,5 @@
         <box size="${base_length} ${tube_width} ${drivebase_total_height}"/>
       </geometry>
-      <origin xyz="0 ${drivebase_beam_width / 2 + tube_width / 2} 0" />
+      <origin xyz="0 ${drivebase_beam_width / 2 + tube_width / 2} 0.1143" />
     </visual>
     <visual>

Commit message: Model updates

File: src/tfr_description/xacro/model_base.xacro (robot description, xacro)
@@ -4,5 +4,5 @@
   <link name="base_footprint" />
   <joint name="base_footprint_joint" type="fixed">
-    <origin xyz="0 0 0.017" rpy="0 0 0" />
+    <origin xyz="0 0 0.07" rpy="0 0 0" />
     <parent link="base_footprint" />
     <child link="base_link" />
@@ -14,5 +14,5 @@
         <box size="${base_length} ${tube_width} ${drivebase_total_height}"/>
       </geometry>
-      <origin xyz="0 ${drivebase_beam_width / 2 + tube_width / 2} 0.1143" />
+      <origin xyz="0 ${drivebase_beam_width / 2 + tube_width / 2} 0.2243" />
     </visual>
     <visual>
