Commit message: bug for melody to look at

File: src/tfr_description/xacro/model_constants.xacro (robot description, xacro)
@@ -46,6 +46,6 @@
   <xacro:property name="lower_arm_width" value="${82.55*mmtom}" />
   <xacro:property name="lower_arm_height" value="${107.09*mmtom}" /> <!-- Original H: 107.09 mm -->
-  <xacro:property name="lower_arm_min" value="0.104" /> <!-- Not given measures-->
-  <xacro:property name="lower_arm_max" value="1.55" /> <!-- Not given measures-->
+  <xacro:property name="lower_arm_min" value="1.8" /> <!-- Not given measures-->
+  <xacro:property name="lower_arm_max" value="5.1" /> <!-- Not given measures-->
   <!-- Upper arm parameters -->
   <xacro:property name="upper_arm_mass" value="${6.4}"/>

File: src/urdf_files/urdf/urdf_files.urdf (robot description, URDF)
Before this commit: robot urdf_files, 5 links, 4 joints
Joints:
- joint Lower-Arm: limit (none) -> lower=1.8 upper=5.1 effort=1.0 velocity=1.0; type continuous -> revolute
- joint Scoop: limit (none) -> lower=0.3 upper=2.7 effort=1.0 velocity=1.0; type continuous -> revolute
- joint Upper-Arm: limit (none) -> lower=1.1 upper=4.5 effort=1.0 velocity=1.0; type continuous -> revolute

Commit message: Fixing control bug with 0's being sent while moving

File: src/tfr_description/xacro/model_constants.xacro (robot description, xacro)
@@ -46,5 +46,5 @@
   <xacro:property name="lower_arm_width" value="${82.55*mmtom}" />
   <xacro:property name="lower_arm_height" value="${107.09*mmtom}" /> <!-- Original H: 107.09 mm -->
-  <xacro:property name="lower_arm_min" value="0.104" /> <!-- Not given measures-->
+  <xacro:property name="lower_arm_min" value="0.206" /> <!-- Not given measures-->
   <xacro:property name="lower_arm_max" value="1.55" /> <!-- Not given measures-->
   <!-- Upper arm parameters -->
@@ -54,5 +54,5 @@
   <xacro:property name="upper_arm_height" value="${102.94*mmtom}" />
   <xacro:property name="upper_arm_min" value="0.98"/> <!-- Not given measures-->
-  <xacro:property name="upper_arm_max" value="2.4"/> <!-- Not given measures-->
+  <xacro:property name="upper_arm_max" value="1.33"/> <!-- Not given measures-->
   <!-- Scoop parameters -->
   <xacro:property name="scoop_mass" value="${3.6}"/>
@@ -60,6 +60,6 @@
   <xacro:property name="scoop_length" value="${153.16*mmtom}" />
   <xacro:property name="scoop_diameter" value="${157*mmtom}" /> <!-- Not given measures-->
-  <xacro:property name="scoop_min" value="-1.16614" /> <!-- Not given measures-->
-  <xacro:property name="scoop_max" value="1.62" /> <!-- Not given measures-->
+  <xacro:property name="scoop_min" value="-1.65" /> <!-- Not given measures-->
+  <xacro:property name="scoop_max" value="0.25" /> <!-- Not given measures-->
   <!-- Depth 185.42-->
 </robot>

Commit message: Trying to get better performance from Aruco Action Server

File: src/tfr_description/xacro/model_constants.xacro (robot description, xacro)
@@ -46,5 +46,5 @@
   <xacro:property name="lower_arm_width" value="${82.55*mmtom}" />
   <xacro:property name="lower_arm_height" value="${107.09*mmtom}" /> <!-- Original H: 107.09 mm -->
-  <xacro:property name="lower_arm_min" value="0.206" /> <!-- Not given measures-->
+  <xacro:property name="lower_arm_min" value="0.20" /> <!-- Not given measures-->
   <xacro:property name="lower_arm_max" value="1.55" /> <!-- Not given measures-->
   <!-- Upper arm parameters -->
