Commit message: Update model_arm.xacro

File: src/tfr_description/xacro/model_arm.xacro (robot description, xacro)
@@ -7,5 +7,5 @@
         <cylinder radius="${turntable_radius}" length="${turntable_height}" />
       </geometry>
-      <origin xyz="0 0 ${turntable_height/2}" rpy="0 0 ${pi}" />
+      <origin xyz="0 0 ${turntable_height/2}" rpy="0 0 0" />
     </visual>
     <collision>
@@ -13,5 +13,5 @@
         <cylinder radius="${turntable_radius}" length="${turntable_height}" />
       </geometry>
-      <origin xyz="0 0 ${turntable_height/2}" rpy="0 0 ${pi}" />
+      <origin xyz="0 0 ${turntable_height/2}" rpy="0 0 0" />
     </collision>
     <!-- test -->
