Commit message: added joint limits to 2021 urdf

File: src/tfr_description/urdf_2021/urdf/urdf_v2.urdf (robot description, URDF)
Before this commit: robot robot, 6 links, 5 joints
Joints:
- joint Lower-Arm: limit (none) -> lower=-1.2 upper=0.55 effort=1000.0 velocity=0.5; origin xyz=0 0.18949 0 rpy=1.5708 1.0411 1.5708 -> xyz=0 0.18949 0 rpy=1.5708 1 1.5708; type continuous -> revolute
- joint Scoop: limit (none) -> lower=-1.65 upper=0.25 effort=1000.0 velocity=0.5; type continuous -> revolute
- joint Upper-Arm: limit (none) -> lower=0.98 upper=1.33 effort=1000.0 velocity=0.5; type continuous -> revolute
